File: PCB/tpms_silencer.kicad_pcb (KiCad board)
At the start: 2 copper layers, 33 x 51.6 mm, 26 parts, among them J1 AVR-ISP-6, SW1 SW_SPST, U1 ATtiny841-SSU, U2 MICRF112YMM, Y1 8MHz, Y2 9.84375MHz

Commit message: leaf
Parts:
- added REF**: TinkerTown_Silkscreen, !Custom:TinkerTown_Silkscreen, F.Cu at (49.8, 64.6)
- Y1: footprint Crystal:Crystal_SMD_TXC_7A-2Pin_5x3.2mm -> Crystal:Crystal_SMD_5032-2Pin_5.0x3.2mm
- Y2: footprint Crystal:Crystal_SMD_HC49-SD -> Crystal:Crystal_SMD_TXC_AX_8045-2Pin_8.0x4.5mm
Routing:
- net Net-(C4-Pad1): track 13.8 -> 10.9 mm
- net Net-(C5-Pad1): track 15.2 -> 14.2 mm
Other:
- board text added: "TPMS Silencer v3"
- board text removed: "TPMS Silencer v2"
