File: PCB/tpms_silencer.sch (KiCad schematic (older format))
At the start: 25 parts, among them J1 AVR-ISP-6, U1 ATtiny841-SSU, U2 MICRF112YMM, Y1 8MHz, Y2 9.84375MHz

Commit message: Change programming header, comments on capacitor, v2 layout, hole for mounting in enclosure
Parts:
- C6: value 12pF -> 10pF
- J1: footprint Connector_JST:JST_SH_BM06B-SRSS-TB_1x06-1MP_P1.00mm_Vertical -> Connector_PinHeader_2.54mm:PinHeader_2x03_P2.54mm_Vertical_SMD
- Y2: footprint Crystal:Crystal_SMD_TXC_AX_8045-2Pin_8.0x4.5mm -> Crystal:Crystal_SMD_HC49-SD
- gave numbers to parts that had none: 1
Other:
- note added: "10pF gives\n33.5kHz spread"
- note added: "8MHz Internal Oscillator\nmight suffice"
Changed lines of the file:
@@
 P 3900 2550
 F 0 "C6" V 4100 2550 50  0000 C CNN
-F 1 "12pF" V 4000 2500 50  0000 C CNN
+F 1 "10pF" V 4000 2500 50  0000 C CNN
 F 2 "Capacitor_SMD:C_0805_2012Metric" H 3900 2550 50  0001 C CNN
 F 3 "" H 3900 2550 50  0001 C CNN
@@
 F 0 "Y2" V 3754 2038 50  0000 L CNN
 F 1 "9.84375MHz" V 3845 2038 50  0000 L CNN
-F 2 "Crystal:Crystal_SMD_TXC_AX_8045-2Pin_8.0x4.5mm" H 3800 1950 50  0001 C CNN
+F 2 "Crystal:Crystal_SMD_HC49-SD" H 3800 1950 50  0001 C CNN
 F 3 "" H 3800 1950 50  0001 C CNN
 	1    3800 1950
@@
 F 0 "J1" H 950 1900 50  0000 R CNN
 F 1 "AVR-ISP-6" H 1300 1800 50  0000 R CNN
-F 2 "Connector_JST:JST_SH_BM06B-SRSS-TB_1x06-1MP_P1.00mm_Vertical" V 700 1450 50  0001 C CNN
+F 2 "Connector_PinHeader_2.54mm:PinHeader_2x03_P2.54mm_Vertical_SMD" V 700 1450 50  0001 C CNN
 F 3 "" H -325 850 50  0001 L CNN
 	1    950  1400
@@
 Wire Wire Line
 	5800 1950 6050 1950
-$Comp
-L Device:R_Small R?
+Wire Wire Line
+	2550 4900 2550 5000
+$Comp
+L power:VDD #PWR017
+U 1 1 5BE8D2F4
+P 2800 5000
+F 0 "#PWR017" H 2800 4850 50  0001 C CNN
+F 1 "VDD" H 2817 5173 50  0000 C CNN
+F 2 "" H 2800 5000 50  0001 C CNN
+F 3 "" H 2800 5000 50  0001 C CNN
+	1    2800 5000
+	1    0    0    -1
+$EndComp
+Text Notes 3700 2800 0    50   ~ 0
+10pF gives\n33.5kHz spread
+Wire Notes Line
+	2900 4300 2900 5350
+Wire Notes Line
+	2900 5350 3600 5350
+Wire Notes Line
+	3600 5350 3600 4300
+Wire Notes Line
+	3600 4300 2900 4300
+Text Notes 2850 5550 0    50   ~ 0
+8MHz Internal Oscillator\nmight suffice
+Wire Wire Line
+	2800 5350 2800 5000
+Wire Wire Line
+	2550 5350 2800 5350
+Wire Wire Line
+	2550 5200 2550 5350
+$Comp
+L Device:R_Small R1
 U 1 1 5BE8BD48
 P 2550 5100
-F 0 "R?" H 2609 5146 50  0000 L CNN
+F 0 "R1" H 2609 5146 50  0000 L CNN
 F 1 "100k" H 2609 5055 50  0000 L CNN
 F 2 "Resistor_SMD:R_0805_2012Metric" H 2550 5100 50  0001 C CNN
@@
 	1    0    0    -1
 $EndComp
-Wire Wire Line
-	2550 4900 2550 5000
-$Comp
-L power:VDD #PWR?
-U 1 1 5BE8D2F4
-P 2800 5000
-F 0 "#PWR?" H 2800 4850 50  0001 C CNN
-F 1 "VDD" H 2817 5173 50  0000 C CNN
-F 2 "" H 2800 5000 50  0001 C CNN
-F 3 "" H 2800 5000 50  0001 C CNN
-	1    2800 5000
-	1    0    0    -1
-$EndComp
-Wire Wire Line
-	2550 5200 2550 5350
-Wire Wire Line
-	2550 5350 2800 5350
-Wire Wire Line
-	2800 5350 2800 5000
 $EndSCHEMATC

Commit message: V2 - sent for fab.
Parts:
- added SW1: SW_SPST, Button_Switch_SMD:SW_SPST_PTS645, symbol Switch:SW_SPST
- J1: footprint Connector_PinHeader_2.54mm:PinHeader_2x03_P2.54mm_Vertical_SMD -> !Custom:AVR-SMD-Programming-Header
- Y1: footprint Crystal:Crystal_SMD_HC49-SD -> Crystal:Crystal_SMD_TXC_7A-2Pin_5x3.2mm
Connections:
- wire segments 70 -> 75
- no-connect marks 3 -> 2
Changed lines of the file:
@@
 encoding utf-8
 Sheet 1 1
-Title "CalmTPMS"
+Title "TPMS Silencer"
 Date ""
-Rev "v1"
+Rev "v2"
 Comp ""
 Comment1 ""
@@
 F 0 "J1" H 950 1900 50  0000 R CNN
 F 1 "AVR-ISP-6" H 1300 1800 50  0000 R CNN
-F 2 "Connector_PinHeader_2.54mm:PinHeader_2x03_P2.54mm_Vertical_SMD" V 700 1450 50  0001 C CNN
+F 2 "!Custom:AVR-SMD-Programming-Header" V 700 1450 50  0001 C CNN
 F 3 "" H -325 850 50  0001 L CNN
 	1    950  1400
@@
 F 0 "Y1" V 3054 4788 50  0000 L CNN
 F 1 "8MHz" V 3145 4788 50  0000 L CNN
-F 2 "Crystal:Crystal_SMD_HC49-SD" H 3100 4700 50  0001 C CNN
+F 2 "Crystal:Crystal_SMD_TXC_7A-2Pin_5x3.2mm" H 3100 4700 50  0001 C CNN
 F 3 "" H 3100 4700 50  0001 C CNN
 	1    3100 4700
@@
 	1    0    0    -1
 $EndComp
-NoConn ~ 2400 4400
 NoConn ~ 2400 4800
 $Comp
@@
 	1    0    0    -1
 $EndComp
+$Comp
+L Switch:SW_SPST SW1
+U 1 1 5BF1F002
+P 3250 4150
+F 0 "SW1" H 3250 4385 50  0000 C CNN
+F 1 "SW_SPST" H 3250 4294 50  0000 C CNN
+F 2 "Button_Switch_SMD:SW_SPST_PTS645" H 3250 4150 50  0001 C CNN
+F 3 "" H 3250 4150 50  0001 C CNN
+	1    3250 4150
+	1    0    0    -1
+$EndComp
+Wire Wire Line
+	2400 4400 2850 4400
+Wire Wire Line
+	2850 4400 2850 4150
+Wire Wire Line
+	2850 4150 3050 4150
+Wire Wire Line
+	3450 4150 3750 4150
+Wire Wire Line
+	3750 4150 3750 4450
+$Comp
+L power:GNDREF #PWR018
+U 1 1 5BF26970
+P 3750 4450
+F 0 "#PWR018" H 3750 4200 50  0001 C CNN
+F 1 "GNDREF" H 3755 4277 50  0000 C CNN
+F 2 "" H 3750 4450 50  0001 C CNN
+F 3 "" H 3750 4450 50  0001 C CNN
+	1    3750 4450
+	1    0    0    -1
+$EndComp

Commit message: Prep for release.
Other:
- moved on the sheet: BT1
Changed lines of the file:
@@
 EESchema Schematic File Version 4
-LIBS:tpms_silencer-cache
-EELAYER 26 0
+EELAYER 29 0
 EELAYER END
 $Descr A4 11693 8268
@@
 L Device:Battery_Cell BT1
 U 1 1 5BBDAE9A
-P 2000 1100
-F 0 "BT1" H 2118 1196 50  0000 L CNN
-F 1 "CR2032" H 2118 1105 50  0000 L CNN
-F 2 "Battery:BatteryHolder_Keystone_3034_1x20mm" V 2000 1160 50  0001 C CNN
-F 3 "~" V 2000 1160 50  0001 C CNN
-	1    2000 1100
+P 2000 1200
+F 0 "BT1" H 2118 1296 50  0000 L CNN
+F 1 "CR2032" H 2118 1205 50  0000 L CNN
+F 2 "Battery:BatteryHolder_Keystone_3034_1x20mm" V 2000 1260 50  0001 C CNN
+F 3 "~" V 2000 1260 50  0001 C CNN
+	1    2000 1200
 	1    0    0    -1
 $EndComp
@@
 L power:VDD #PWR0101
 U 1 1 5BBDB4FE
-P 2000 900
-F 0 "#PWR0101" H 2000 750 50  0001 C CNN
-F 1 "VDD" H 2017 1073 50  0000 C CNN
-F 2 "" H 2000 900 50  0001 C CNN
-F 3 "" H 2000 900 50  0001 C CNN
-	1    2000 900
+P 2000 1000
+F 0 "#PWR0101" H 2000 850 50  0001 C CNN
+F 1 "VDD" H 2017 1173 50  0000 C CNN
+F 2 "" H 2000 1000 50  0001 C CNN
+F 3 "" H 2000 1000 50  0001 C CNN
+	1    2000 1000
 	1    0    0    -1
 $EndComp
@@
 L power:GNDREF #PWR0102
 U 1 1 5BBDB53B
-P 2000 1200
-F 0 "#PWR0102" H 2000 950 50  0001 C CNN
-F 1 "GNDREF" H 2005 1027 50  0000 C CNN
-F 2 "" H 2000 1200 50  0001 C CNN
-F 3 "" H 2000 1200 50  0001 C CNN
-	1    2000 1200
-	1    0    0    -1
-$EndComp
+P 2000 1300
+F 0 "#PWR0102" H 2000 1050 50  0001 C CNN
+F 1 "GNDREF" H 2005 1127 50  0000 C CNN
+F 2 "" H 2000 1300 50  0001 C CNN
+F 3 "" H 2000 1300 50  0001 C CNN
+	1    2000 1300
+	1    0    0    -1
+$EndComp

Commit message: notes for 433mhz parts
Other:
- note added: "(13.560MHz)"
- note added: "(3.9pF)"
- note added: "(433.92MHz in parenthesis)"
- note added: "(82nH)"
- note added: "(NP)"
Changed lines of the file:
@@
 EESchema Schematic File Version 4
+LIBS:tpms_silencer-cache
 EELAYER 29 0
 EELAYER END
@@
 	1    0    0    -1
 $EndComp
+Text Notes 3900 2100 0    50   ~ 0
+(13.560MHz)
+Text Notes 8100 2350 0    50   ~ 0
+(82nH)
+Text Notes 8600 2750 0    50   ~ 0
+(3.9pF)
+Text Notes 7150 1750 0    50   ~ 0
+(NP)
+Text Notes 4900 1350 0    50   ~ 0
+(433.92MHz in parenthesis)
 $EndSCHEMATC

Commit message: leaf
Parts:
- Y1: footprint Crystal:Crystal_SMD_TXC_7A-2Pin_5x3.2mm -> Crystal:Crystal_SMD_5032-2Pin_5.0x3.2mm
- Y2: footprint Crystal:Crystal_SMD_HC49-SD -> Crystal:Crystal_SMD_TXC_AX_8045-2Pin_8.0x4.5mm
Changed lines of the file:
@@
 F 0 "Y2" V 3754 2038 50  0000 L CNN
 F 1 "9.84375MHz" V 3845 2038 50  0000 L CNN
-F 2 "Crystal:Crystal_SMD_HC49-SD" H 3800 1950 50  0001 C CNN
+F 2 "Crystal:Crystal_SMD_TXC_AX_8045-2Pin_8.0x4.5mm" H 3800 1950 50  0001 C CNN
 F 3 "" H 3800 1950 50  0001 C CNN
 	1    3800 1950
@@
 F 0 "Y1" V 3054 4788 50  0000 L CNN
 F 1 "8MHz" V 3145 4788 50  0000 L CNN
-F 2 "Crystal:Crystal_SMD_TXC_7A-2Pin_5x3.2mm" H 3100 4700 50  0001 C CNN
+F 2 "Crystal:Crystal_SMD_5032-2Pin_5.0x3.2mm" H 3100 4700 50  0001 C CNN
 F 3 "" H 3100 4700 50  0001 C CNN
 	1    3100 4700
